File: template-module/template-module.kicad_sch (KiCad schematic)
At the start: 3 parts, among them J1 SEAF-20-01-X-10-X-RA-GP-X-XX

Commit message: upload
Parts:
- added R3, R4: 120R, symbol Device:R_Small
Connections:
- net CAN_H: now also R3.2
- net CAN_L: now also R4.2
- net GND: now also J1.F6, J1.F8, J1.G10, J1.G12, J1.G14, J1.G16, J1.G19, J1.G2, J1.G20, J1.G4, J1.G6, J1.G8, J1.H12, J1.H3, J1.H6, J1.H9
- net at J1.F5: now also R3.1
- net at J1.F7: now also R4.1
- net PCIE0_TXP: now reaches J1.G1
- net PCIE1_TXN: now reaches J1.G11
- net PCIE1_RXP: now reaches J1.G13
- net PCIE1_RXN: now reaches J1.G15
- net USB_DP: now reaches J1.G17
- net USB_DM: now reaches J1.G18
- net PCIE0_TXN: now reaches J1.G3
- net PCIE0_RXP: now reaches J1.G5
- net PCIE0_RXN: now reaches J1.G7
- net PCIE1_TXP: now reaches J1.G9
- net ETH0_TXP: now reaches J1.H1
- net ETH1_RXP: now reaches J1.H10
- net ETH1_RXN: now reaches J1.H11
- net ETH0_TXN: now reaches J1.H2
- net ETH0_RXP: now reaches J1.H4
- net ETH0_RXN: now reaches J1.H5
- net ETH1_TXP: now reaches J1.H7
- net ETH1_TXN: now reaches J1.H8

Commit message: upload
Connections:
- net GND: now also J1.H15, J1.H18, J1.H19, J1.H20, J1.I1, J1.I12, J1.I15, J1.I18, J1.I20, J1.I4, J1.I7, J1.I9
- net MIPS0_CLKN: now reaches J1.I10
- net MIPS0_DL1_DP: now reaches J1.I11
- net MIPS0_DL1_DN: now reaches J1.I13
- net MIPS0_DL2_DP: now reaches J1.I14
- net MIPS0_DL2_DN: now reaches J1.I16
- net MIPS0_I2C_SDA: now reaches J1.I17
- net MIPS0_I2C_SCL: now reaches J1.I19
- net SYS_WAKE: now reaches J1.I2
- net SYS_RST: now reaches J1.I3
- net MOD_ID_SDA: now reaches J1.I5
- net MOD_ID_SCL: now reaches J1.I6
- net MIPS0_CLKP: now reaches J1.I8
- net SATA_TXP: now reaches J1.H13
- net SATA_TXN: now reaches J1.H14
- net SATA_RXP: now reaches J1.H16
- net SATA_RXN: now reaches J1.H17
- no-connect marks 0 -> 60
Other:
- note added: "3V3 PDS"
- note added: "5V PDS"
- note added: "CAM"
- note added: "CAN BUS"
- note added: "ETHERNET"
- note added: "GND"
- note added: "I2C0"
- note added: "IFS"
- note added: "PCIE X2"
- note added: "RESERVED"
- note added: "SATA"
- note added: "SPI0"
- note added: "To WC Mux"
- note added: "UART0"
- note added: "USB"
